File: ExtruderControlBoard2209/ExtruderControlBoard2209.kicad_pcb (KiCad board)
At the start: 2 copper layers, 42.7 x 62 mm, 83 parts, among them J10 USB_B, J15 Conn_Stepper, J17 Power_In, J2 Conn_Heater, J6 ICSP, Q1 Q_NMOS_GDS, Q2 Q_NMOS_GSD, Q3 Q_NMOS_GSD, SW1 SW_RESET, U1 MP1584EN-LF-Z, U2 ATmega328P-AU, U3 TMC2209-LA, U4 CH330N, U5 USBLC6-2SC6, Y1 Resonator

Commit message: emifix
Parts:
- removed I2C: Conn_I2C, Connector_PinHeader_2.54mm:PinHeader_1x02_P2.54mm_Vertical
- removed Spread: SPREAD, Jumper:SolderJumper-3_P1.3mm_Open_RoundedPad1.0x1.5mm_NumberLabels
- added C19: 100nF, Capacitor_SMD:C_0805_2012Metric_Pad1.18x1.45mm_HandSolder, B.Cu at (150.7, 83.8)
- added I2C1: Conn_I2C, Connector_PinHeader_2.54mm:PinHeader_1x02_P2.54mm_Vertical, F.Cu at (167.8, 75.8)
- AUX1: renamed from Diag CS
- C11, R12, R13: moved to F.Cu
- C5: footprint Capacitor_SMD:CP_Elec_6.3x7.7 -> Capacitor_SMD:CP_Elec_4x5.4
- D4: moved to B.Cu
- J8: renamed from USB   Buck
- J9: renamed from Servo V  G
- moved C18 20.7 mm to (169.8, 43.2), turned to 270 degrees
- moved Heater1 17.0 mm to (141.9, 38.7), turned to 180 degrees
- moved C11 13.9 mm to (165.2, 55.4), turned to 180 degrees
- moved C3 13.8 mm to (151.7, 65.8)
- moved R13 12.8 mm to (150.9, 73.1), turned to 315 degrees
- moved F1 11.6 mm to (144.4, 47.2), turned to 180 degrees
- moved AUX1 11.1 mm to (162.8, 66.2)
- moved D4 10.5 mm to (145.3, 44.1)
- moved C4 10.1 mm to (157.2, 77.7), turned to 270 degrees
- moved D5 9.57 mm to (158.2, 62.2), turned to 270 degrees
- moved C5 9.50 mm to (166.2, 49.8), turned to 270 degrees
- moved C14 9.38 mm to (135.8, 49.7), turned to 270 degrees
- moved R12 9.25 mm to (153.2, 72.1)
- moved U1 8.95 mm to (150.4, 59.6)
- moved R17 7.81 mm to (145.8, 57.3), turned to 90 degrees
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- renumbered B to FB30R1, Met_Det to FS1, J2 to Heater1, J6 to ICSP1, Probe to J12, J15 to Motor1, J17 to Power1, TH to TH1
Connections:
- Heater1 pad 1: Net-(J2-Pad1) -> 24VHeater
- Heater1 pad 2: 24VHeater -> Net-(Heater1-Pad2)
- Q1 pad 2: Net-(J2-Pad1) -> Net-(Heater1-Pad2)
- U3 pad 7: SPREAD -> Net-(U3-Pad7)
Routing:
- net GND: track 90.9 -> 28.6 mm, vias 31 -> 54
- net TX_MCU: track 20.5 -> 51.4 mm, vias 2 -> 0
- net RX_MCU: track 19.7 -> 48.8 mm
- net SPREAD: track 24.6 -> 0.00 mm, vias 2 -> 0
- net +5V: track 163.2 -> 140.0 mm, vias 7 -> 6
- net +24V: track 119.4 -> 97.1 mm
- net M_RX: track 37.2 -> 22.7 mm
- net Diag: track 17.3 -> 30.6 mm, vias 0 -> 1
- net A_CS: track 26.7 -> 13.9 mm, vias 1 -> 0
- net SDA: track 24.9 -> 12.5 mm, vias 1 -> 0
- net 5V_BUCK: track 28.2 -> 40.1 mm
- net Net-(C4-Pad1): track 2.52 -> 13.9 mm
- net MT_DET: track 18.4 -> 7.86 mm, vias 2 -> 0
- net LED: track 45.4 -> 55.2 mm, vias 2 -> 0
- net Heater_PWM: track 42.8 -> 51.6 mm, vias 2 -> 0
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- added copper zone on B.Cu, net +5V
- added copper zone on F.Cu, net +5V
Other:
- board text added: "+"
- board text added: "-"
- board text added: "Diag CS"
- board text added: "ExtruderController 2209 REV 1.1"
- board text added: "Probe"
- board text added: "SDA SCL"
- board text added: "Servo V G"
- board text added: "USB DCDC"
- board text removed: "ExtruderController 2209 V1"
- board text removed: "SCL SDA"

Commit message: minor optimization
Parts:
- added C20: 100nF, Capacitor_SMD:C_0805_2012Metric_Pad1.18x1.45mm_HandSolder, B.Cu at (151.5, 67.3)
- R14, R15: footprint Resistor_SMD:R_0805_2012Metric_Pad1.20x1.40mm_HandSolder -> Resistor_SMD:R_1206_3216Metric_Pad1.30x1.75mm_HandSolder
- moved C3 3.73 mm to (148.1, 64.9)
- moved R15 0.10 mm to (153.4, 92.3)
Routing:
- net Net-(C20-Pad2): track 0.00 -> 4.17 mm
- net +5V: track 140.0 -> 137.4 mm
- net Net-(R15-Pad2): track 4.28 -> 3.35 mm
- net Net-(R14-Pad2): track 4.28 -> 3.49 mm
