File: ExtruderControlBoard2209/ExtruderControlBoard2209.sch (KiCad schematic (older format))
At the start: 79 parts, among them J1 Conn_TH, J10 USB_B, J11 A_CS, J12 Conn_Probe, J15 Conn_Stepper, J17 Power_In, J2 Conn_Heater, J3 Conn_Fan1, J4 Conn_MT_DET, J5 Conn_I2C, J6 ICSP, J7 Conn_Fan2, J8 PowerSelection, J9 Conn_Servo, Q1 Q_NMOS_GDS, Q2 Q_NMOS_GSD, Q3 Q_NMOS_GSD, SW1 SW_RESET, U1 MP1584EN-LF-Z, U2 ATmega328P-AU, U3 TMC2209-LA, U4 CH330N, U5 USBLC6-2SC6, Y1 Resonator

Commit message: emifix
Parts:
- removed JP1: SPREAD, Jumper:SolderJumper-3_P1.3mm_Open_RoundedPad1.0x1.5mm_NumberLabels, symbol Jumper:SolderJumper_3_Open
- added C19: 100nF, Capacitor_SMD:C_0805_2012Metric_Pad1.18x1.45mm_HandSolder, symbol Device:C
- C5: footprint Capacitor_SMD:CP_Elec_6.3x7.7 -> Capacitor_SMD:CP_Elec_4x5.4
- renumbered J11 to AUX1, J4 to FS1, J3 to Fan1, J7 to Fan2, J2 to Heater1, J5 to I2C1, J6 to ICSP1, J15 to Motor1, J17 to Power1, J1 to TH1
Connections:
- net +5V: now also C19.2
- net 24VHeater: now also Heater1.1 (Pin_1); no longer Heater1.2 (Pin_2)
- net GND: now also C19.1
- net at Q1.2 (D): now also Heater1.2 (Pin_2); no longer Heater1.1 (Pin_1)
- net SPREAD: no longer names the net of U3.7 (SPREAD)
- no-connect marks 8 -> 9
Other:
- moved on the sheet: Heater1
Changed lines of the file:
@@
 TX_MCU
 $Comp
-L Connector_Generic:Conn_02x03_Odd_Even J6
+L Connector_Generic:Conn_02x03_Odd_Even ICSP1
 U 1 1 615FDF9E
 P 4300 1050
-F 0 "J6" H 4350 1367 50  0000 C CNN
+F 0 "ICSP1" H 4350 1367 50  0000 C CNN
 F 1 "ICSP" H 4350 1276 50  0000 C CNN
 F 2 "Connector_PinHeader_2.54mm:PinHeader_2x03_P2.54mm_Vertical" H 4300 1050 50  0001 C CNN
@@
 $EndComp
 $Comp
-L Connector:Conn_01x04_Male J15
+L Connector:Conn_01x04_Male Motor1
 U 1 1 6156DA06
 P 5400 1850
-F 0 "J15" H 5372 1732 50  0000 R CNN
+F 0 "Motor1" H 5372 1732 50  0000 R CNN
 F 1 "Conn_Stepper" H 5372 1823 50  0000 R CNN
 F 2 "Connector_JST:JST_XH_B4B-XH-A_1x04_P2.50mm_Vertical" H 5400 1850 50  0001 C CNN
@@
 Connection ~ 1750 7600
 $Comp
-L Connector:Conn_01x02_Male J3
+L Connector:Conn_01x02_Male Fan1
 U 1 1 616B1002
 P 2600 7200
-F 0 "J3" H 2708 7381 50  0000 C CNN
+F 0 "Fan1" H 2708 7381 50  0000 C CNN
 F 1 "Conn_Fan1" H 2708 7290 50  0000 C CNN
 F 2 "Connector_JST:JST_XH_B2B-XH-A_1x02_P2.50mm_Vertical" H 2600 7200 50  0001 C CNN
@@
 Connection ~ 3500 7600
 $Comp
-L Connector:Conn_01x02_Male J7
+L Connector:Conn_01x02_Male Fan2
 U 1 1 616BC085
 P 4350 7200
-F 0 "J7" H 4458 7381 50  0000 C CNN
+F 0 "Fan2" H 4458 7381 50  0000 C CNN
 F 1 "Conn_Fan2" H 4458 7290 50  0000 C CNN
 F 2 "Connector_JST:JST_XH_B2B-XH-A_1x02_P2.50mm_Vertical" H 4350 7200 50  0001 C CNN
@@
 $EndComp
 $Comp
-L Connector:Conn_01x02_Male J1
+L Connector:Conn_01x02_Male TH1
 U 1 1 61751E8B
 P 850 6500
-F 0 "J1" H 958 6681 50  0000 C CNN
+F 0 "TH1" H 958 6681 50  0000 C CNN
 F 1 "Conn_TH" H 958 6590 50  0000 C CNN
 F 2 "Connector_JST:JST_XH_B2B-XH-A_1x02_P2.50mm_Vertical" H 850 6500 50  0001 C CNN
@@
 Connection ~ 1350 6800
 $Comp
-L Connector:Conn_01x03_Male J4
+L Connector:Conn_01x03_Male FS1
 U 1 1 6180A3F6
 P 3000 5700
-F 0 "J4" H 3108 5981 50  0000 C CNN
+F 0 "FS1" H 3108 5981 50  0000 C CNN
 F 1 "Conn_MT_DET" H 3108 5890 50  0000 C CNN
 F 2 "Connector_JST:JST_XH_B3B-XH-A_1x03_P2.50mm_Vertical" H 3000 5700 50  0001 C CNN
@@
 DIR
 $Comp
-L Connector:Conn_01x02_Male J5
+L Connector:Conn_01x02_Male I2C1
 U 1 1 6184BF26
 P 2550 1050
-F 0 "J5" H 2658 1231 50  0000 C CNN
+F 0 "I2C1" H 2658 1231 50  0000 C CNN
 F 1 "Conn_I2C" H 2658 1140 50  0000 C CNN
 F 2 "Connector_PinHeader_2.54mm:PinHeader_1x02_P2.54mm_Vertical" H 2550 1050 50  0001 C CNN
@@
 MT_DET
 $Comp
-L Connector:Conn_01x02_Male J17
+L Connector:Conn_01x02_Male Power1
 U 1 1 617474FE
 P 700 900
-F 0 "J17" V 762 944 50  0000 L CNN
+F 0 "Power1" V 762 944 50  0000 L CNN
 F 1 "Power_In" V 853 944 50  0000 L CNN
 F 2 "TerminalBlock_Phoenix:TerminalBlock_Phoenix_MKDS-1,5-2_1x02_P5.00mm_Horizontal" H 700 900 50  0001 C CNN
@@
 F 0 "C5" H 6800 700 50  0000 R CNN
 F 1 "220UF/16V" H 6950 600 50  0000 R CNN
-F 2 "Capacitor_SMD:CP_Elec_6.3x7.7" H 6688 700 50  0001 C CNN
+F 2 "Capacitor_SMD:CP_Elec_4x5.4" H 6688 700 50  0001 C CNN
 F 3 "~" H 6650 850 50  0001 C CNN
 	1    6650 850
@@
 	0    1    1    0
 $EndComp
-Wire Wire Line
-	1150 7300 1150 7350
-Wire Wire Line
-	1050 7300 1150 7300
-$Comp
-L Connector:Conn_01x02_Male J2
+$Comp
+L Connector:Conn_01x02_Male Heater1
 U 1 1 6164A2AB
-P 850 7200
-F 0 "J2" H 958 7381 50  0000 C CNN
-F 1 "Conn_Heater" H 958 7290 50  0000 C CNN
-F 2 "TerminalBlock_Phoenix:TerminalBlock_Phoenix_MKDS-1,5-2_1x02_P5.00mm_Horizontal" H 850 7200 50  0001 C CNN
-F 3 "~" H 850 7200 50  0001 C CNN
-	1    850  7200
+P 850 7100
+F 0 "Heater1" H 958 7281 50  0000 C CNN
+F 1 "Conn_Heater" H 958 7190 50  0000 C CNN
+F 2 "TerminalBlock_Phoenix:TerminalBlock_Phoenix_MKDS-1,5-2_1x02_P5.00mm_Horizontal" H 850 7100 50  0001 C CNN
+F 3 "~" H 850 7100 50  0001 C CNN
+	1    850  7100
 	1    0    0    -1
 $EndComp
@@
 F 3 "http://www.wch.cn/downloads/file/240.html" H 8050 3450 50  0001 C CNN
 	1    8400 2650
-	1    0    0    -1
-$EndComp
-$Comp
-L ExtruderControlBoard2209-rescue:TMC2209-LA-Tmc2209 U3
-U 1 1 616473A0
-P 4250 2750
-F 0 "U3" H 5250 3137 60  0000 C CNN
-F 1 "TMC2209-LA" H 5250 3031 60  0000 C CNN
-F 2 "Tmc2209:TMC2209-LA" H 5250 2990 60  0001 C CNN
-F 3 "" H 4250 2750 60  0000 C CNN
-	1    4250 2750
 	1    0    0    -1
 $EndComp
@@
 $EndComp
 Connection ~ 3950 4050
-Connection ~ 4250 4050
 $Comp
 L power:+24V #PWR0107
@@
 	1    4250 2950
 	0    1    1    0
-$EndComp
-$Comp
-L Jumper:SolderJumper_3_Open JP1
-U 1 1 619D9778
-P 4400 2050
-F 0 "JP1" H 4400 2255 50  0000 C CNN
-F 1 "SPREAD" H 4400 2164 50  0000 C CNN
-F 2 "Jumper:SolderJumper-3_P1.3mm_Open_RoundedPad1.0x1.5mm_NumberLabels" H 4400 2050 50  0001 C CNN
-F 3 "~" H 4400 2050 50  0001 C CNN
-	1    4400 2050
-	1    0    0    -1
-$EndComp
-Text GLabel 4250 3350 0    50   Input ~ 0
-SPREAD
-Text GLabel 4400 2200 3    50   UnSpc ~ 0
-SPREAD
-$Comp
-L power:+5V #PWR0110
-U 1 1 619E0945
-P 4200 2050
-F 0 "#PWR0110" H 4200 1900 50  0001 C CNN
-F 1 "+5V" V 4215 2178 50  0000 L CNN
-F 2 "" H 4200 2050 50  0001 C CNN
-F 3 "" H 4200 2050 50  0001 C CNN
-	1    4200 2050
-	0    -1   -1   0
-$EndComp
-$Comp
-L power:GND #PWR0111
-U 1 1 619E2B26
-P 4600 2050
-F 0 "#PWR0111" H 4600 1800 50  0001 C CNN
-F 1 "GND" V 4605 1922 50  0000 R CNN
-F 2 "" H 4600 2050 50  0001 C CNN
-F 3 "" H 4600 2050 50  0001 C CNN
-	1    4600 2050
-	0    -1   -1   0
 $EndComp
 NoConn ~ 4250 3550
@@
 U 1 1 61C3CA09
 P 10200 5450
-F 0 "C12" H 10250 5350 50  0000 L CNN
+F 0 "C12" H 9950 5350 50  0000 L CNN
 F 1 "100nF" H 10100 5350 50  0000 L CNN
 F 2 "Capacitor_SMD:C_0805_2012Metric_Pad1.18x1.45mm_HandSolder" H 10238 5300 50  0001 C CNN
@@
 	4800 5150 4800 5250
 $Comp
-L Connector:Conn_01x04_Male J11
+L Connector:Conn_01x04_Male AUX1
 U 1 1 61BA5167
 P 6050 7000
-F 0 "J11" H 6158 7281 50  0000 C CNN
+F 0 "AUX1" H 6158 7281 50  0000 C CNN
 F 1 "A_CS" H 6158 7190 50  0000 C CNN
 F 2 "Connector_PinHeader_2.54mm:PinHeader_1x04_P2.54mm_Vertical" H 6050 7000 50  0001 C CNN
@@
 Wire Wire Line
 	6050 1150 6200 1150
-Text GLabel 1150 7350 3    50   Input ~ 0
+Text GLabel 1050 7100 2    50   Input ~ 0
 24VHeater
 Text GLabel 8000 4250 1    50   Input ~ 0
@@
 U 1 1 61A759E8
 P 10050 5900
-F 0 "C11" H 10165 5946 50  0000 L CNN
-F 1 "100nf" H 10165 5855 50  0000 L CNN
+F 0 "C11" H 9850 6000 50  0000 L CNN
+F 1 "100nf" H 9700 5900 50  0000 L CNN
 F 2 "Capacitor_SMD:C_0805_2012Metric_Pad1.18x1.45mm_HandSolder" H 10088 5750 50  0001 C CNN
 F 3 "~" H 10050 5900 50  0001 C CNN
@@
 Wire Wire Line
 	6250 6900 6550 6900
+NoConn ~ 4250 3350
+Connection ~ 4250 4050
+$Comp
+L Device:C C19
+U 1 1 6206ED18
+P 6250 4300
+F 0 "C19" V 5998 4300 50  0000 C CNN
+F 1 "100nF" V 6089 4300 50  0000 C CNN
+F 2 "Capacitor_SMD:C_0805_2012Metric_Pad1.18x1.45mm_HandSolder" H 6288 4150 50  0001 C CNN
+F 3 "~" H 6250 4300 50  0001 C CNN
+	1    6250 4300
+	-1   0    0    1
+$EndComp
+$Comp
+L ExtruderControlBoard2209-rescue:TMC2209-LA-Tmc2209 U3
+U 1 1 616473A0
+P 4250 2750
+F 0 "U3" H 5250 3137 60  0000 C CNN
+F 1 "TMC2209-LA" H 5250 3031 60  0000 C CNN
+F 2 "Tmc2209:TMC2209-LA" H 5250 2990 60  0001 C CNN
+F 3 "" H 4250 2750 60  0000 C CNN
+	1    4250 2750
+	1    0    0    -1
+$EndComp
+Connection ~ 6250 4150
+$Comp
+L power:GND #PWR033
+U 1 1 62082C47
+P 6250 4450
+F 0 "#PWR033" H 6250 4200 50  0001 C CNN
+F 1 "GND" H 6255 4277 50  0000 C CNN
+F 2 "" H 6250 4450 50  0001 C CNN
+F 3 "" H 6250 4450 50  0001 C CNN
+	1    6250 4450
+	1    0    0    -1
+$EndComp
 $EndSCHEMATC

Commit message: minor optimization
Parts:
- added C20: 100nF, Capacitor_SMD:C_0805_2012Metric_Pad1.18x1.45mm_HandSolder, symbol Device:C
- R14, R15: footprint Resistor_SMD:R_0805_2012Metric_Pad1.20x1.40mm_HandSolder -> Resistor_SMD:R_1206_3216Metric_Pad1.30x1.75mm_HandSolder
Connections:
- net GND: now also C20.1
- net at U2.20 (AREF): now also C20.2
- no-connect marks 9 -> 8
Changed lines of the file:
@@
 Wire Wire Line
 	900  1000 1000 1000
-NoConn ~ 800  2450
 $Comp
 L power:PWR_FLAG #FLG0102
@@
 F 0 "R14" V 6593 2950 50  0000 C CNN
 F 1 "0R11" V 6684 2950 50  0000 C CNN
-F 2 "Resistor_SMD:R_0805_2012Metric_Pad1.20x1.40mm_HandSolder" V 6730 2950 50  0001 C CNN
+F 2 "Resistor_SMD:R_1206_3216Metric_Pad1.30x1.75mm_HandSolder" V 6730 2950 50  0001 C CNN
 F 3 "~" H 6800 2950 50  0001 C CNN
 	1    6800 2950
@@
 F 0 "R15" V 6593 3350 50  0000 C CNN
 F 1 "0R11" V 6684 3350 50  0000 C CNN
-F 2 "Resistor_SMD:R_0805_2012Metric_Pad1.20x1.40mm_HandSolder" V 6730 3350 50  0001 C CNN
+F 2 "Resistor_SMD:R_1206_3216Metric_Pad1.30x1.75mm_HandSolder" V 6730 3350 50  0001 C CNN
 F 3 "~" H 6800 3350 50  0001 C CNN
 	1    6800 3350
@@
 	1    0    0    -1
 $EndComp
+$Comp
+L Device:C C20
+U 1 1 61C5B1C7
+P 650 2200
+F 0 "C20" H 765 2246 50  0000 L CNN
+F 1 "100nF" H 765 2155 50  0000 L CNN
+F 2 "Capacitor_SMD:C_0805_2012Metric_Pad1.18x1.45mm_HandSolder" H 688 2050 50  0001 C CNN
+F 3 "~" H 650 2200 50  0001 C CNN
+	1    650  2200
+	1    0    0    -1
+$EndComp
+Wire Wire Line
+	800  2450 650  2450
+Wire Wire Line
+	650  2450 650  2350
+$Comp
+L power:GND #PWR034
+U 1 1 61C661C9
+P 650 2050
+F 0 "#PWR034" H 650 1800 50  0001 C CNN
+F 1 "GND" H 655 1877 50  0000 C CNN
+F 2 "" H 650 2050 50  0001 C CNN
+F 3 "" H 650 2050 50  0001 C CNN
+	1    650  2050
+	-1   0    0    1
+$EndComp
 $EndSCHEMATC
